File: sram.kicad_sch (KiCad schematic)
At the start: 4 parts, among them U1 STM32H753ZIT6, U2 IS61WV204816BLL-10TLI

Commit message: add SDIO
Connections:
- net GND: now also U2.7 (CS#)
- net ~{CS}: no longer names the net of U1.97 (FMC_NE1)
- net ~{CS}: no longer U2.7 (CS#)
- no-connect marks 3 -> 4
Changed lines of the file:
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@@
+	)
+	(junction
+		(at 189.23 80.01)
+		(diameter 0)
+		(color 0 0 0 0)
 	)
 	(junction
@@
 	)
 	(no_connect
+		(at 100.33 31.75)
+	)
+	(no_connect
 		(at 191.77 95.25)
 	)
@@
 	)
 	(bus_entry
-		(at 179.07 67.31)
-		(size 2.54 -2.54)
-		(stroke
-			(width 0)
-			(type default)
-		)
-	)
-	(bus_entry
 		(at 234.95 69.85)
 		(size -2.54 -2.54)
@@
 	)
 	(bus_entry
-		(at 109.22 31.75)
-		(size 2.54 2.54)
-		(stroke
-			(width 0)
-			(type default)
-		)
-	)
-	(bus_entry
 		(at 109.22 102.87)
 		(size 2.54 2.54)
@@
 	(bus
 		(pts
-			(xy 111.76 34.29) (xy 111.76 36.83)
+			(xy 111.76 27.94) (xy 111.76 36.83)
 		)
 		(stroke
@@
 		)
 	)
-	(bus
-		(pts
-			(xy 111.76 27.94) (xy 111.76 34.29)
-		)
-		(stroke
-			(width 0)
-			(type default)
-		)
-	)
 	(wire
 		(pts
@@
 		)
 	)
-	(wire
-		(pts
-			(xy 181.61 64.77) (xy 191.77 64.77)
-		)
-		(stroke
-			(width 0)
-			(type default)
-		)
-	)
 	(bus
 		(pts
@@
 	(bus
 		(pts
-			(xy 179.07 62.23) (xy 179.07 67.31)
+			(xy 179.07 62.23) (xy 179.07 69.85)
 		)
 		(stroke
@@
 		)
 	)
-	(bus
-		(pts
-			(xy 179.07 67.31) (xy 179.07 69.85)
-		)
-		(stroke
-			(width 0)
-			(type default)
-		)
-	)
 	(wire
 		(pts
@@
 		)
 	)
+	(wire
+		(pts
+			(xy 189.23 64.77) (xy 189.23 80.01)
+		)
+		(stroke
+			(width 0)
+			(type default)
+		)
+	)
 	(bus
 		(pts
@@
 		)
 	)
-	(wire
-		(pts
-			(xy 100.33 31.75) (xy 109.22 31.75)
-		)
-		(stroke
-			(width 0)
-			(type default)
-		)
-	)
 	(bus
 		(pts
@@
 	(wire
 		(pts
-			(xy 165.1 80.01) (xy 191.77 80.01)
+			(xy 165.1 80.01) (xy 189.23 80.01)
 		)
 		(stroke
@@
 	(wire
 		(pts
+			(xy 191.77 64.77) (xy 189.23 64.77)
+		)
+		(stroke
+			(width 0)
+			(type default)
+		)
+	)
+	(wire
+		(pts
 			(xy 232.41 69.85) (xy 222.25 69.85)
 		)
@@
 		(pts
 			(xy 100.33 77.47) (xy 109.22 77.47)
+		)
+		(stroke
+			(width 0)
+			(type default)
+		)
+	)
+	(wire
+		(pts
+			(xy 189.23 80.01) (xy 191.77 80.01)
 		)
 		(stroke
@@
 		)
 	)
-	(label "~{CS}"
-		(at 182.88 64.77 0)
-		(fields_autoplaced yes)
-		(effects
-			(font
-				(size 1.27 1.27)
-			)
-			(justify left bottom)
-		)
-	)
 	(label "D7"
 		(at 182.88 90.17 0)
@@
 		(fields_autoplaced yes)
 		(effects
-			(font
-				(size 1.27 1.27)
-			)
-			(justify right bottom)
-		)
-	)
-	(label "~{CS}"
-		(at 107.95 31.75 180)
-		(fields_autoplaced yes)
-		(effects

Commit message: checkpoint
Connections:
- net A0: now also U2.5 (A0)
- net A1: no longer U2.5 (A0)
Changed lines of the file:
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@@
 	(wire
 		(pts
-			(xy 165.1 87.63) (xy 165.1 80.01)
+			(xy 165.1 86.36) (xy 165.1 80.01)
 		)
 		(stroke
@@
 		)
 	)
+	(wire
+		(pts
+			(xy 100.33 95.25) (xy 109.22 95.25)
+		)
+		(stroke
+			(width 0)
+			(type default)
+		)
+	)
 	(bus
 		(pts
@@
 		(pts
 			(xy 179.07 90.17) (xy 179.07 92.71)
-		)
-		(stroke
-			(width 0)
-			(type default)
-		)
-	)
-	(wire
-		(pts
-			(xy 100.33 95.25) (xy 109.22 95.25)
 		)
 		(stroke
@@
 		)
 	)
-	(label "SRAM{~{CS}, ~{WE}, ~{OE}, A[0..20], ~{UB}, ~{LB}, D[0..15]}"
+	(label "{~{CS}, ~{WE}, ~{OE}, A[0..20], ~{UB}, ~{LB}, D[0..15]}"
 		(at 123.19 152.4 0)
 		(fields_autoplaced yes)
@@
 		)
 	)
-	(label "A1"
+	(label "A0"
 		(at 182.88 59.69 0)
 		(fields_autoplaced yes)
@@
 	(symbol
 		(lib_id "power:GND")
-		(at 165.1 87.63 0)
+		(at 165.1 86.36 0)
 		(unit 1)
 		(exclude_from_sim no)
@@
 		(fields_autoplaced yes)
 		(property "Reference" "#PWR03"
-			(at 165.1 93.98 0)
+			(at 165.1 92.71 0)
 			(effects
 				(font
@@
 		)
 		(property "Value" "GND"
-			(at 165.1 92.71 0)
+			(at 165.1 91.44 0)
 			(effects
 				(font
@@
 		)
 		(property "Footprint" ""
-			(at 165.1 87.63 0)
+			(at 165.1 86.36 0)
 			(effects
 				(font
@@
 		)
 		(property "Datasheet" ""
-			(at 165.1 87.63 0)
+			(at 165.1 86.36 0)
 			(effects
 				(font
@@
 		)
 		(property "Description" "Power symbol creates a global label with name \"GND\" , ground"
-			(at 165.1 87.63 0)
+			(at 165.1 86.36 0)
 			(effects
 				(font
