File: unused.kicad_sch (KiCad schematic)
At the start: 1 part, among them U1 STM32H753ZIT6

Commit message: checkpoint
Changed lines of the file:
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@@
 	)
 	(symbol
+		(lib_name "STM32H753ZITx_1")
 		(lib_id "stm32h753:STM32H753ZITx")
 		(at 104.14 105.41 0)
