File: stm32simh.kicad_pcb (KiCad board)
At the start: 4 copper layers, 0 parts

Commit message: first stab at board layout
Parts:
- added C1: 0.1uF, Capacitor_SMD:C_0402_1005Metric, F.Cu at (118.0, 57.0)
- added C10: 0.1uF, Capacitor_SMD:C_0402_1005Metric, F.Cu at (161.5, 64.2)
- added C11: 0.1uF, Capacitor_SMD:C_0402_1005Metric, F.Cu at (156.2, 57.0)
- added C12: 0.1uF, Capacitor_SMD:C_0402_1005Metric, F.Cu at (145.2, 57.0)
- added C13: 0.1uF, Capacitor_SMD:C_0402_1005Metric, F.Cu at (149.7, 57.0)
- added C14: 0.1uF, Capacitor_SMD:C_0402_1005Metric, F.Cu at (139.8, 57.0)
- added C15: 0.1uF, Capacitor_SMD:C_0402_1005Metric, F.Cu at (136.0, 66.2)
- added C16: 0.1uF, Capacitor_SMD:C_0402_1005Metric, F.Cu at (136.2, 78.8)
- added C17: 0.1uF, Capacitor_SMD:C_0402_1005Metric, F.Cu at (147.0, 82.5)
- added C18: 0.1uF, Capacitor_SMD:C_0402_1005Metric, F.Cu at (151.5, 82.5)
- added C19: 0.1uF, Capacitor_SMD:C_0402_1005Metric, F.Cu at (157.5, 82.5)
- added C2: 0.1uF, Capacitor_SMD:C_0402_1005Metric, F.Cu at (118.5, 81.0)
- added C20: 4.7uF, Capacitor_SMD:C_0805_2012Metric, F.Cu at (162.2, 83.8)
- added C21: 0.1uF, Capacitor_SMD:C_0402_1005Metric, F.Cu at (162.2, 62.8)
- added C22: 1uF, Capacitor_SMD:C_0402_1005Metric, F.Cu at (162.2, 61.8)
- added C23: 2.2uF, Capacitor_SMD:C_0603_1608Metric, F.Cu at (133.0, 77.9)
- added C24: 2.2uF, Capacitor_SMD:C_0603_1608Metric, F.Cu at (141.0, 56.5)
- added C25: 4.7µF, Capacitor_SMD:C_0805_2012Metric, F.Cu at (171.8, 65.8)
- added C26: 0.1µF, Capacitor_SMD:C_0402_1005Metric, F.Cu at (171.0, 67.5)
- added C27: 0.1µF, Capacitor_SMD:C_0402_1005Metric, F.Cu at (169.2, 66.5)
- added C28: 4.7µF, Capacitor_SMD:C_0805_2012Metric, F.Cu at (168.0, 64.2)
- added C29: 10µF 16V, Capacitor_SMD:C_0603_1608Metric, F.Cu at (130.5, 51.0)
- added C3: 500nF, Capacitor_SMD:C_0402_1005Metric, F.Cu at (114.4, 93.6)
- added C30: 0.1uF, Capacitor_SMD:C_0402_1005Metric, F.Cu at (147.4, 44.2)
- added C31: 0.1uF, Capacitor_SMD:C_0402_1005Metric, F.Cu at (147.2, 41.2)
- added C32: 4.7uF, Capacitor_SMD:C_0805_2012Metric, F.Cu at (146.8, 36.9)
- added C33: 0.1uF, Capacitor_SMD:C_0402_1005Metric, F.Cu at (156.5, 42.0)
- added C34: 470pF, Capacitor_SMD:C_0402_1005Metric, F.Cu at (152.2, 46.3)
- added C35: 1uF, Capacitor_SMD:C_0402_1005Metric, F.Cu at (152.2, 47.4)
- added C36: 10µF 16V, Capacitor_SMD:C_0603_1608Metric, F.Cu at (177.4, 55.6)
- added C37: 22µF 25V, Capacitor_SMD:C_0805_2012Metric, F.Cu at (180.9, 48.1)
- added C38: 34pF, Capacitor_SMD:C_0402_1005Metric, F.Cu at (145.6, 48.9)
- added C39: 34pF, Capacitor_SMD:C_0402_1005Metric, F.Cu at (148.9, 50.7)
- added C4: 0.1uF, Capacitor_SMD:C_0402_1005Metric, F.Cu at (166.0, 82.0)
- added C5: 0.1uF, Capacitor_SMD:C_0402_1005Metric, F.Cu at (149.8, 89.8)
- added C6: 4.7uF, Capacitor_SMD:C_0805_2012Metric, F.Cu at (150.2, 93.0)
- added C7: 1pF, Capacitor_SMD:C_0402_1005Metric, F.Cu at (164.5, 77.0)
- added C8: 1pF, Capacitor_SMD:C_0402_1005Metric, F.Cu at (162.8, 77.5)
- added C9: 0.1uF, Capacitor_SMD:C_0402_1005Metric, F.Cu at (161.5, 70.8)
- added D1: 30V 100mA, Diode_SMD:D_0603_1608Metric, F.Cu at (157.3, 89.5)
- added D2: GRN, Diode_SMD:D_0603_1608Metric, F.Cu at (167.8, 76.5)
- added D3: GRN, Diode_SMD:D_0603_1608Metric, F.Cu at (169.5, 76.5)
- added D4: SP0503BAHT, Package_TO_SOT_SMD:SOT-143, F.Cu at (174.7, 73.5)
- added D5: GRN, Diode_SMD:D_0603_1608Metric, F.Cu at (150.5, 102.8)
- added D6: GRN, Diode_SMD:D_0603_1608Metric, F.Cu at (186.3, 61.6)
- added D7: GRN, Diode_SMD:D_0603_1608Metric, F.Cu at (182.1, 36.6)
- added J1: Micro_SD_Card_Det_Hirose_DM3AT, Connector_Card:microSD_HC_Hirose_DM3AT-SF-PEJM5, F.Cu at (141.0, 95.5)
- added J2: ARM JTAG, Package_SO:SOIC-10_3.9x4.9mm_P1mm, F.Cu at (119.8, 95.6)
- added J3: USB_C_USB2.0_16P, Connector_USB:USB_C_Receptacle_HCTL_HC-TYPE-C-16P-01A, F.Cu at (184.5, 70.5)
- added J4: SERIAL1, Connector_PinHeader_2.54mm:PinHeader_1x03_P2.54mm_Vertical, F.Cu at (186.5, 88.3)
- added J5: RJ45, Connector_RJ:RJ45_Amphenol_RJMG1BD3B8K1ANR, F.Cu at (127.4, 43.9)
- added L1: 33Ω @ 100MHz 400mA 240mΩ, Inductor_SMD:L_0402_1005Metric, F.Cu at (182.9, 62.9)
- added L2: 33Ω @ 100MHz 400mA 240mΩ, Inductor_SMD:L_0402_1005Metric, F.Cu at (144.9, 45.5)
- added L3: 2.2µH 70MHz+ 1A+ 0.5Ω-, Inductor_SMD:L_Taiyo-Yuden_NR-24xx, F.Cu at (177.4, 48.9)
- added R1: 15k, Resistor_SMD:R_0402_1005Metric, F.Cu at (166.0, 80.9)
- added R11: 5.1k, Resistor_SMD:R_0402_1005Metric, F.Cu at (181.4, 76.6)
- added R12: 5.1k, Resistor_SMD:R_0402_1005Metric, F.Cu at (181.4, 64.6)
- added R13: 15k, Resistor_SMD:R_0402_1005Metric, F.Cu at (152.2, 101.5)
- added R14: 12.1k, Resistor_SMD:R_0402_1005Metric, F.Cu at (144.9, 43.5)
- added R15: 49.9 1/4W+, Resistor_SMD:R_0805_2012Metric, F.Cu at (136.1, 41.7)
- added R16: 49.9 1/4W+, Resistor_SMD:R_0805_2012Metric, F.Cu at (136.1, 46.5)
- added R17: 49.9 1/4W+, Resistor_SMD:R_0805_2012Metric, F.Cu at (136.1, 39.3)
- added R18: 49.9 1/4W+, Resistor_SMD:R_0805_2012Metric, F.Cu at (136.1, 44.1)
- added R19: 100, Resistor_SMD:R_0402_1005Metric, F.Cu at (135.0, 34.8)
- added R2: 15k, Resistor_SMD:R_0402_1005Metric, F.Cu at (131.5, 91.5)
- added R20: 100, Resistor_SMD:R_0402_1005Metric, F.Cu at (135.0, 36.0)
- added R21: 33k, Resistor_SMD:R_0402_1005Metric, F.Cu at (181.4, 61.9)
- added R22: 47k, Resistor_SMD:R_0402_1005Metric, F.Cu at (175.2, 53.4)
- added R23: 15k, Resistor_SMD:R_0402_1005Metric, F.Cu at (181.6, 38.4)
- added R24: 100, Resistor_SMD:R_0402_1005Metric, F.Cu at (147.2, 39.0)
- added R25: 100, Resistor_SMD:R_0402_1005Metric, F.Cu at (147.2, 40.2)
- added R26: 100, Resistor_SMD:R_0402_1005Metric, F.Cu at (154.2, 56.2)
- added R27: 100, Resistor_SMD:R_0402_1005Metric, F.Cu at (153.2, 56.2)
- added R28: 100, Resistor_SMD:R_0402_1005Metric, F.Cu at (155.2, 56.2)
- added R3: 15k, Resistor_SMD:R_0402_1005Metric, F.Cu at (131.5, 93.8)
- added R4: 15k, Resistor_SMD:R_0402_1005Metric, F.Cu at (131.5, 95.0)
- added R5: 15k, Resistor_SMD:R_0402_1005Metric, F.Cu at (131.5, 90.2)
- added R6: 15k, Resistor_SMD:R_0402_1005Metric, F.Cu at (131.5, 88.0)
- added R7: 15k, Resistor_SMD:R_0402_1005Metric, F.Cu at (166.2, 76.5)
- added R8: 15k, Resistor_SMD:R_0402_1005Metric, F.Cu at (171.0, 76.5)
- added R9: 15k, Resistor_SMD:R_0402_1005Metric, F.Cu at (165.4, 70.0)
- added U1: STM32H753ZIT6, Package_QFP:LQFP-144_20x20mm_P0.5mm, F.Cu at (148.8, 69.8)
- added U2: IS61WV204816BLL-10TLI, SOP50P2000X120-48N:SOP50P2000X120-48N, F.Cu at (118.5, 69.1)
- added U3: LAN8720A, Package_DFN_QFN:VQFN-24-1EP_4x4mm_P0.5mm_EP2.5x2.5mm, F.Cu at (151.3, 42.4)
- added U4: CP2102N, CP2102N-QFN:CP2102N-QFN20, F.Cu at (168.8, 70.2)
- added U5: LM3671 3.3V, Package_TO_SOT_SMD:TSOT-23-5, F.Cu at (177.4, 52.6)
- added V1: CR2032, Battery:BatteryHolder_Keystone_1060_1x2032, F.Cu at (170.8, 96.2)
- added Y1: ABS06W-32.768kHz-D-2-T DISC, Crystal:Crystal_SMD_2012-2Pin_2.0x1.2mm, F.Cu at (163.2, 75.5)
- added Y3: 25MHz, Crystal:Crystal_SMD_3225-4Pin_3.2x2.5mm, F.Cu at (148.3, 48.4)
Routing:
- net /Ethernet/~{RESET}: track 0.00 -> 118.3 mm, vias 0 -> 2
- net GND: track 0.00 -> 91.7 mm, vias 0 -> 77
- net +3.3V: track 0.00 -> 81.2 mm, vias 0 -> 34
- net Net-(J5-RCT): track 0.00 -> 62.8 mm, vias 0 -> 5
- net /SRAM/~{UB}: track 0.00 -> 57.6 mm, vias 0 -> 2
- net /SRAM/A5: track 0.00 -> 57.1 mm, vias 0 -> 2
- net /SRAM/~{LB}: track 0.00 -> 56.4 mm, vias 0 -> 2
- net /SRAM/A4: track 0.00 -> 54.8 mm, vias 0 -> 2
- net /SRAM/A6: track 0.00 -> 54.5 mm, vias 0 -> 2
- net /SRAM/A20: track 0.00 -> 54.2 mm, vias 0 -> 2
- net /SRAM/A3: track 0.00 -> 54.0 mm, vias 0 -> 2
- net /SRAM/A2: track 0.00 -> 53.2 mm, vias 0 -> 2
- net /SRAM/A1: track 0.00 -> 52.6 mm, vias 0 -> 2
- net /SRAM/A7: track 0.00 -> 52.1 mm, vias 0 -> 2
- net /SRAM/A0: track 0.00 -> 51.8 mm, vias 0 -> 2
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- added copper zone on F.Cu, net +3.3V
- added copper zone on In2.Cu, net +3.3V
- added copper zone on F.Cu, net GND
- added copper zone on In1.Cu, net GND
Other:
- board outline added: 78.8 x 75.6 mm
